Commit message: Keep AR2010/D500 meshes unmodified (no collision-hull swap) (#1)
* Keep ROS-Industrial meshes unmodified and stop swapping collision hulls

Visual STLs were already byte-identical to motoman noetic-devel; the URDF
converter had rewritten collision paths onto those visual files. Vendor the
original collision hulls separately, never render them, and SHA-256-check
the copies in CI so they cannot be silently decimated.

Co-authored-by: MQCIA <MQCIA@users.noreply.github.com>

* Add a local Verbotics inventory agent for the Windows install

Cloud agents cannot read C:\Program Files\Verbotics Weld 2026. The PowerShell
wrapper runs on that PC, unpacks .vbmodel zips, and writes inventory.json plus
extracted model.json (torch TCP) for the cloud agent to consume.

Co-authored-by: MQCIA <MQCIA@users.noreply.github.com>

* Add full Verbotics dump tooling and record cloud placement miss

Self-hosted worker verbotics-pc is required for C:\ access; this commit
ships verbotics_full_dump.py / updated PS1 and an inventory noting the
Linux cloud host cannot see the install.

Co-authored-by: MQCIA <MQCIA@users.noreply.github.com>

* Fix Verbotics Windows dump launcher and document PC-hosted agent flow

The PowerShell wrapper now discovers install roots reliably and invokes
verbotics_full_dump.py with matching flags. Docs clarify that this cloud chat
cannot jump onto verbotics-pc — start a new agent with that environment, or run
the dump locally and commit from-verbotics/.

Co-authored-by: MQCIA <MQCIA@users.noreply.github.com>

* Document full Verbotics dump via local script or PC-hosted agent

Clarify that this cloud chat cannot jump onto verbotics-pc; dump the whole
install with the PowerShell launcher or start a new agent on that machine.

Co-authored-by: MQCIA <MQCIA@users.noreply.github.com>

---------

Co-authored-by: Cursor Agent <cursoragent@cursor.com>
Co-authored-by: MQCIA <MQCIA@users.noreply.github.com>

File: frontend/public/models/ar2010/ar2010.urdf (robot description, URDF)
Before this commit: robot ar2010, 10 links, 9 joints
Links:
- link base_link: geometry collision mesh filename=collision/base_link.stl; visual mesh filename=visual/base_link.stl
- link link_1_s: geometry collision mesh filename=collision/link_1_s.stl; visual mesh filename=visual/link_1_s.stl
- link link_2_l: geometry collision mesh filename=collision/link_2_l.stl; visual mesh filename=visual/link_2_l.stl
- link link_3_u: geometry collision mesh filename=collision/link_3_u.stl; visual mesh filename=visual/link_3_u.stl
- link link_4_r: geometry collision mesh filename=collision/link_4_r.stl; visual mesh filename=visual/link_4_r.stl
- link link_5_b: geometry collision mesh filename=collision/link_5_b.stl; visual mesh filename=visual/link_5_b.stl
- link link_6_t: geometry collision mesh filename=collision/link_6_t.stl; visual mesh filename=visual/link_6_t.stl

File: frontend/public/models/motopos_d500/motopos_d500.urdf (robot description, URDF)
Before this commit: robot motopos_d500, 5 links, 4 joints
Links:
- link base_link: geometry collision mesh filename=collision/base_link.stl; visual mesh filename=visual/base_link.stl
- link link_1: geometry collision mesh filename=collision/link_1.stl; visual mesh filename=visual/link_1.stl
- link link_2: geometry collision mesh filename=collision/link_2.stl; visual mesh filename=visual/link_2.stl
