Commit message: Add ROS-I flange link to MA2010 URDF
Match AR2010: flange at 100 mm from link_6_t, tool0 coincident with
flange, so the torch parent resolves to the mechanical face.

Co-authored-by: MQCIA <MQCIA@users.noreply.github.com>

File: frontend/public/models/ma2010/ma2010.urdf (robot description, URDF)
Before this commit: robot ma2010, 9 links, 8 joints
Links:
- added link flange
Joints:
- removed joint joint_6_t-tool0
- added joint flange-tool0: type fixed, parent flange, child tool0, origin xyz=0 0 0 rpy=0 0 0
- added joint joint_6_t-flange: type fixed, parent link_6_t, child flange, origin xyz=0.100 0 0 rpy=0 0 0
